Commit message: Fix the laser joint

File: src/bumperbot_description/urdf/bumperbot.urdf.xacro (robot description, xacro)
@@ -201,5 +201,5 @@
   </link>
   <joint name="laser_joint" type="fixed">
-    <origin xyz="-0.0050526 -0.0023221 0.1208" rpy="0 0 3.14" />
+    <origin xyz="-0.0050526 -0.0023221 0.1208" rpy="0 0 -1.5708" />
     <parent link="base_link" />
     <child link="laser_link" />

Commit message: UPdate to burgerbot description

File: src/bumperbot_description/urdf/bumperbot.urdf.xacro (robot description, xacro)
@@ -206,4 +206,44 @@
     <axis xyz="0 0 0" />
   </joint>
+  <link name="camera_link">
+    <inertial>
+      <origin xyz="0 0 0" rpy="0 0 0" />
+      <mass value="0.05" />
+      <inertia ixx="1.0E-6" ixy="0" ixz="0" iyy="1.0E-6" iyz="0" izz="1.0E-6" />
+    </inertial>
+    <visual>
+      <origin xyz="0 0 0" rpy="0 0 0" />
+      <geometry>
+        <box size="0.03 0.03 0.03" />
+      </geometry>
+      <material name="black"/>
+    </visual>
+    <collision>
+      <origin xyz="0 0 0" rpy="0 0 0" />
+      <geometry>
+        <box size="0.03 0.03 0.03" />
+      </geometry>
+    </collision>
+  </link>
+  <!-- Mounted on the front of the robot, directly above the front caster (matching
+       caster_front_joint's x/y), 7 inches (0.1778 m) above the ground. base_link
+       already sits 0.033 m above the ground per base_joint, so the offset here is
+       0.1778 - 0.033 = 0.1448 m. -->
+  <joint name="camera_joint" type="fixed">
+    <origin xyz="0.04755 0 0.1448" rpy="0 0 0" />
+    <parent link="base_link" />
+    <child link="camera_link" />
+  </joint>
+  <!-- usb_cam/ros2_aruco publish in the standard camera optical frame convention
+       (Z out of the lens, X right, Y down), not the robot convention (X forward,
+       Y left, Z up) used everywhere else here. This fixed rotation is the standard
+       REP103-to-optical-frame conversion, and "default_cam" matches the exact
+       frame_id ros2_aruco is already publishing poses in. -->
+  <link name="default_cam"/>
+  <joint name="camera_optical_joint" type="fixed">
+    <origin xyz="0 0 0" rpy="-1.5707963267948966 0 -1.5707963267948966" />
+    <parent link="camera_link" />
+    <child link="default_cam" />
+  </joint>
   <material name="blue">
     <color rgba="0 0 1 1"/>

Commit message: Visual mesh fixes for the robot

File: src/bumperbot_description/urdf/bumperbot.urdf.xacro (robot description, xacro)
@@ -19,5 +19,5 @@
     </inertial>
     <visual>
-      <origin xyz="0 0 0" rpy="0 0 0" />
+      <origin xyz="0 0 0" rpy="-1.5707963267948966 0 0" />
       <geometry>
         <mesh filename="package://bumperbot_description/meshes/base_link.STL" />
@@ -26,5 +26,5 @@
     </visual>
     <collision>
-      <origin xyz="0 0 0" rpy="0 0 0" />
+      <origin xyz="0 0 0" rpy="-1.5707963267948966 0 0" />
       <geometry>
         <mesh filename="package://bumperbot_description/meshes/base_link.STL" />
@@ -46,5 +46,5 @@
     </inertial>
     <visual>
-      <origin xyz="0 0 0" rpy="1.57 0 0" />
+      <origin xyz="0 0 0" rpy="0 0 0" />
       <geometry>
         <mesh filename="package://bumperbot_description/meshes/wheel_right_link.STL" />
@@ -75,5 +75,5 @@
     </inertial>
     <visual>
-      <origin xyz="0 0 0" rpy="-1.57 0 0" />
+      <origin xyz="0 0 0" rpy="-3.14159265358979 0 0" />
       <geometry>
         <mesh filename="package://bumperbot_description/meshes/wheel_left_link.STL" />
@@ -103,5 +103,5 @@
     </inertial>
     <visual>
-      <origin xyz="0 0 0" rpy="0 0 0" />
+      <origin xyz="0 0 0" rpy="-1.5707963267948966 0 0" />
       <geometry>
         <mesh filename="package://bumperbot_description/meshes/caster_front_link.STL" />
@@ -131,5 +131,5 @@
     </inertial>
     <visual>
-      <origin xyz="0 0 0" rpy="0 0 0" />
+      <origin xyz="0 0 0" rpy="-1.5707963267948966 0 0" />
       <geometry>
         <mesh filename="package://bumperbot_description/meshes/caster_rear_link.STL" />
@@ -187,5 +187,5 @@
     </inertial>
     <visual>
-      <origin xyz="0 0 0" rpy="0 0 0" />
+      <origin xyz="0 0 0" rpy="-1.5707963267948966 0 0" />
       <geometry>
         <mesh filename="package://bumperbot_description/meshes/laser_link.STL" />
@@ -194,5 +194,5 @@
     </visual>
     <collision>
-      <origin xyz="0 0 0" rpy="0 0 0" />
+      <origin xyz="0 0 0" rpy="-1.5707963267948966 0 0" />
       <geometry>
         <mesh filename="package://bumperbot_description/meshes/laser_link.STL" />

Commit message: Bring the camera down more so its correct

File: src/bumperbot_description/urdf/bumperbot.urdf.xacro (robot description, xacro)
@@ -159,5 +159,5 @@
     </inertial>
     <visual>
-      <origin xyz="0 0 0" rpy="0 0 0" />
+      <origin xyz="0 0 0" rpy="-1.5707963267948966 0 0" />
       <geometry>
         <mesh filename="package://bumperbot_description/meshes/imu_link.STL" />
@@ -166,5 +166,5 @@
     </visual>
     <collision>
-      <origin xyz="0 0 0" rpy="0 0 0" />
+      <origin xyz="0 0 0" rpy="-1.5707963267948966 0 0" />
       <geometry>
         <mesh filename="package://bumperbot_description/meshes/imu_link.STL" />
@@ -231,5 +231,5 @@
        0.1778 - 0.033 = 0.1448 m. -->
   <joint name="camera_joint" type="fixed">
-    <origin xyz="0.04755 0 0.1448" rpy="0 0 0" />
+    <origin xyz="0.04755 0 0.0813" rpy="0 0 0" />
     <parent link="base_link" />
     <child link="camera_link" />
